Commit message: latest version in Turtlebot

File: common/asus_xtion_pro.urdf.xacro (robot description, xacro)
@@ -9,6 +9,6 @@
   <xacro:property name="asus_xtion_pro_cam_rel_rgb_py"   value="-0.0220" />
   <!-- Parameterised in part by the values in turtlebot_properties.urdf.xacro -->
-  <!--<xacro:macro name="sensor_asus_xtion_pro" params="parent">
-    <joint name="camera_rgb_joint" type="fixed">
+  <xacro:macro name="sensor_asus_xtion_pro" params="parent">
+    <!--<joint name="camera_rgb_joint" type="fixed">
       <origin xyz="${cam_px} ${asus_xtion_pro_cam_py} ${cam_pz}"
               rpy="${cam_or} ${cam_op} ${cam_oy}"/>
@@ -17,10 +17,4 @@
     </joint>
     <link name="camera_rgb_frame"/>-->
-    <joint name="camera_rgb_joint" type="fixed">
-      <origin xyz="0.00 0.00 0.06" rpy="0 0 0" />
-      <parent link="head_tilt_link"/>
-      <child link="camera_rgb_link" />
-    </joint>
-    <link name="camera_rgb_link" />
     <joint name="camera_rgb_optical_joint" type="fixed">
       <origin xyz="0 0 0" rpy="${-M_PI/2} 0 ${-M_PI/2}" />

File: common/kobuki.urdf.xacro (robot description, xacro)
@@ -209,5 +209,5 @@
     </link>
     <!-- head pan_tilt -->
-    <joint name="head_pan_joint" type="continuous">
+    <joint name="head_pan_joint" type="fixed">
       <origin xyz="-0.20 0.00 0.90" rpy="0 0 0" />
       <parent link="base_link"/>
@@ -215,5 +215,5 @@
     </joint>
     <link name="head_pan_link" />
-    <joint name="head_tilt_joint" type="continuous">
+    <joint name="head_tilt_joint" type="fixed">
       <origin xyz="0.00 0.00 0.05" rpy="0 0 0" />
       <parent link="head_pan_link"/>
@@ -221,4 +221,10 @@
     </joint>
     <link name="head_tilt_link" />
+    <link name="camera_rgb_frame" />
+    <joint name="camera_rgb_joint" type="fixed">
+      <origin xyz="0.00 0.00 0.06" rpy="0 0 0" />
+      <parent link="head_tilt_link"/>
+      <child link="camera_rgb_frame" />
+    </joint>
     <!-- Kobuki Gazebo simulation details -->
     <kobuki_sim/>
