Commit message: camera_rgb_frame added

File: common/kobuki.urdf.xacro (robot description, xacro)
@@ -209,16 +209,16 @@
     </link>
     <!-- head pan_tilt -->
+    <joint name="head_pan_joint" type="continuous">
+      <origin xyz="-0.20 0.00 0.90" rpy="0 0 0" />
+      <parent link="base_link"/>
+      <child link="head_pan_link" />
+    </joint>
     <link name="head_pan_link" />
-    <joint name="head_pan_joint" type="fixed">
-      <origin xyz="0.00 0.00 0.00" rpy="0 0 0" />
-      <parent link="base_link"/>
-      <child link="head_pan_link" />
-    </joint>
-    <link name="head_tilt_link" />
-    <joint name="head_tilt_joint" type="fixed">
-      <origin xyz="0.00 0.00 0.00" rpy="0 0 0" />
+    <joint name="head_tilt_joint" type="continuous">
+      <origin xyz="0.00 0.00 0.05" rpy="0 0 0" />
       <parent link="head_pan_link"/>
       <child link="head_tilt_link" />
     </joint>
+    <link name="head_tilt_link" />
     <!-- Kobuki Gazebo simulation details -->
     <kobuki_sim/>

Commit message: visual link information added

File: common/kobuki.urdf.xacro (robot description, xacro)
@@ -209,4 +209,15 @@
     </link>
     <!-- head pan_tilt -->
+    <link name="head_pan_link" />
+      <visual>
+        <geometry>
+          <box size="0.045 0.03 0.035"/>
+        </geometry>
+        <origin xyz="-0.20 0.00 0.90" rpy="0 0 0" />
+        <material name="blue">
+            <color rgba="0 0 0.8 1"/>
+        </material>
+      </visual>
+    </link>
     <joint name="head_pan_joint" type="fixed">
       <origin xyz="-0.20 0.00 0.90" rpy="0 0 0" />
@@ -214,14 +225,33 @@
       <child link="head_pan_link" />
     </joint>
-    <link name="head_pan_link" />
+    <link name="head_tilt_link" />
+      <visual>
+        <geometry>
+          <box size="0.03 0.035 0.045"/>
+        </geometry>
+        <origin xyz="-0.20 0.00 0.935" rpy="0 0 0" />
+        <material name="blue">
+            <color rgba="0 0 0.8 1"/>
+        </material>
+      </visual>
+    </link>
     <joint name="head_tilt_joint" type="fixed">
-      <origin xyz="0.00 0.00 0.05" rpy="0 0 0" />
+      <origin xyz="0.00 0.00 0.035" rpy="0 0 0" />
       <parent link="head_pan_link"/>
       <child link="head_tilt_link" />
     </joint>
-    <link name="head_tilt_link" />
     <link name="camera_rgb_frame" />
+      <visual>
+        <geometry>
+          <box size="0.025 0.045 0.05"/>
+        </geometry>
+        <origin xyz="-0.20 0.00 0.985" rpy="0 0 0" />
+        <material name="blue">
+            <color rgba="0 0 0.8 1"/>
+        </material>
+      </visual>
+    </link>
     <joint name="camera_rgb_joint" type="fixed">
-      <origin xyz="0.00 0.00 0.06" rpy="0 0 0" />
+      <origin xyz="0.00 0.00 0.05" rpy="0 0 0" />
       <parent link="head_tilt_link"/>
       <child link="camera_rgb_frame" />

Commit message: latest version in Turtlebot

File: common/kobuki.urdf.xacro (robot description, xacro)
@@ -209,10 +209,26 @@
     </link>
     <!-- head pan_tilt -->
-    <link name="head_pan_link" />
+    <link name="head_pan_link">
       <visual>
         <geometry>
           <box size="0.045 0.03 0.035"/>
         </geometry>
-        <origin xyz="-0.20 0.00 0.90" rpy="0 0 0" />
+        <origin xyz="0.0 0.0 -0.035" rpy="0 0 0" />
+        <material name="black">
+            <color rgba="0 0 0 1"/>
+        </material>
+      </visual>
+    </link>
+    <joint name="head_pan_joint" type="fixed">
+      <origin xyz="-0.20 0.00 0.90" rpy="0 0 0" />
+      <parent link="base_link"/>
+      <child link="head_pan_link" />
+    </joint>
+    <link name="head_tilt_link">
+      <visual>
+        <geometry>
+          <box size="0.03 0.035 0.045"/>
+        </geometry>
+        <origin xyz="0.0 0.0 -0.045" rpy="0 0 0" />
         <material name="blue">
             <color rgba="0 0 0.8 1"/>
@@ -220,33 +236,17 @@
       </visual>
     </link>
-    <joint name="head_pan_joint" type="fixed">
-      <origin xyz="-0.20 0.00 0.90" rpy="0 0 0" />
-      <parent link="base_link"/>
-      <child link="head_pan_link" />
-    </joint>
-    <link name="head_tilt_link" />
-      <visual>
-        <geometry>
-          <box size="0.03 0.035 0.045"/>
-        </geometry>
-        <origin xyz="-0.20 0.00 0.935" rpy="0 0 0" />
-        <material name="blue">
-            <color rgba="0 0 0.8 1"/>
-        </material>
-      </visual>
-    </link>
     <joint name="head_tilt_joint" type="fixed">
-      <origin xyz="0.00 0.00 0.035" rpy="0 0 0" />
+      <origin xyz="0.00 0.00 0.045" rpy="0 0 0" />
       <parent link="head_pan_link"/>
       <child link="head_tilt_link" />
     </joint>
-    <link name="camera_rgb_frame" />
+    <link name="camera_rgb_frame">
       <visual>
         <geometry>
           <box size="0.025 0.045 0.05"/>
         </geometry>
-        <origin xyz="-0.20 0.00 0.985" rpy="0 0 0" />
-        <material name="blue">
-            <color rgba="0 0 0.8 1"/>
+        <origin xyz="0.0 0.0 -0.05" rpy="0 0 0" />
+        <material name="white">
+            <color rgba="1 1 1 1"/>
         </material>
       </visual>

Commit message: latest version in Turtlebot

File: common/kobuki.urdf.xacro (robot description, xacro)
@@ -212,7 +212,7 @@
       <visual>
         <geometry>
-          <box size="0.045 0.03 0.035"/>
-        </geometry>
-        <origin xyz="0.0 0.0 -0.035" rpy="0 0 0" />
+          <box size="0.03 0.035 0.045"/>
+        </geometry>
+        <origin xyz="0.0 0.0 0.0" rpy="0 0 0" />
         <material name="black">
             <color rgba="0 0 0 1"/>
@@ -220,5 +220,7 @@
       </visual>
     </link>
-    <joint name="head_pan_joint" type="fixed">
+    <joint name="head_pan_joint" type="revolute">
+      <axis xyz="0 0 1"/>
+      <limit effort="1000.0" lower="-3.1416" upper="3.1416" velocity="0.5"/>
       <origin xyz="-0.20 0.00 0.90" rpy="0 0 0" />
       <parent link="base_link"/>
@@ -228,23 +230,7 @@
       <visual>
         <geometry>
-          <box size="0.03 0.035 0.045"/>
-        </geometry>
-        <origin xyz="0.0 0.0 -0.045" rpy="0 0 0" />
-        <material name="blue">
-            <color rgba="0 0 0.8 1"/>
-        </material>
-      </visual>
-    </link>
-    <joint name="head_tilt_joint" type="fixed">
-      <origin xyz="0.00 0.00 0.045" rpy="0 0 0" />
-      <parent link="head_pan_link"/>
-      <child link="head_tilt_link" />
-    </joint>
-    <link name="camera_rgb_frame">
-      <visual>
-        <geometry>
           <box size="0.025 0.045 0.05"/>
         </geometry>
-        <origin xyz="0.0 0.0 -0.05" rpy="0 0 0" />
+        <origin xyz="0.0 0.0 0.0" rpy="0 0 0" />
         <material name="white">
             <color rgba="1 1 1 1"/>
@@ -252,6 +238,14 @@
       </visual>
     </link>
+    <joint name="head_tilt_joint" type="revolute">
+      <axis xyz="0 1 0"/>
+      <limit effort="1000.0" lower="-3.1416" upper="3.1416" velocity="0.5"/>
+      <origin xyz="0.00 0.00 0.045" rpy="0 0 0.0" />
+      <parent link="head_pan_link"/>
+      <child link="head_tilt_link" />
+    </joint>
+    <link name="camera_rgb_frame"/>
     <joint name="camera_rgb_joint" type="fixed">
-      <origin xyz="0.00 0.00 0.05" rpy="0 0 0" />
+      <origin xyz="0.0 0.0 0.05" rpy="0 0 0" />
       <parent link="head_tilt_link"/>
       <child link="camera_rgb_frame" />

Commit message: head model fixed

File: common/kobuki.urdf.xacro (robot description, xacro)
@@ -209,8 +209,8 @@
     </link>
     <!-- head pan_tilt -->
-    <link name="head_pan_link">
-      <visual>
-        <geometry>
-          <box size="0.03 0.035 0.045"/>
+    <link name="head_base_link">
+      <visual>
+        <geometry>
+          <box size="0.045 0.03 0.035"/>
         </geometry>
         <origin xyz="0.0 0.0 0.0" rpy="0 0 0" />
@@ -220,9 +220,25 @@
       </visual>
     </link>
+    <joint name="head_base_joint" type="fixed">
+      <origin xyz="-0.20 0.00 0.90" rpy="0 0 0" />
+      <parent link="base_link"/>
+      <child link="head_base_link" />
+    </joint>
+    <link name="head_pan_link">
+      <visual>
+        <geometry>
+          <box size="0.03 0.035 0.045"/>
+        </geometry>
+        <origin xyz="0.0 0.0 0.0" rpy="0 0 0" />
+        <material name="blue">
+            <color rgba="0 0 0.8 1"/>
+        </material>
+      </visual>
+    </link>
     <joint name="head_pan_joint" type="revolute">
       <axis xyz="0 0 1"/>
       <limit effort="1000.0" lower="-3.1416" upper="3.1416" velocity="0.5"/>
-      <origin xyz="-0.20 0.00 0.90" rpy="0 0 0" />
-      <parent link="base_link"/>
+      <origin xyz="0.0 0.0 0.035" rpy="0 0 0" />
+      <parent link="head_base_link"/>
       <child link="head_pan_link" />
     </joint>

Commit message: arm model added

File: common/kobuki.urdf.xacro (robot description, xacro)
@@ -208,4 +208,5 @@
       </inertial>
     </link>
+    <!-- FEATURED ROBOT MODEL -->
     <!-- head pan_tilt -->
     <link name="head_base_link">
@@ -267,4 +268,57 @@
       <child link="camera_rgb_frame" />
     </joint>
+    <!-- robot arm as in built as in http://wiki.ros.org/turtlebot_arm -->
+    <link name="arm_base_link">
+      <visual>
+        <geometry>
+          <box size="0.045 0.03 0.035"/>
+        </geometry>
+        <origin xyz="0.0 0.0 0.0" rpy="0 0 0" />
+        <material name="black">
+            <color rgba="0 0 0 1"/>
+        </material>
+      </visual>
+    </link>
+    <joint name="arm_base_joint" type="fixed">
+      <origin xyz="0.10 0.00 0.27" rpy="0 0 0" />
+      <parent link="base_link"/>
+      <child link="arm_base_link" />
+    </joint>
+    <link name="arm_waist_link">
+      <visual>
+        <geometry>
+          <box size="0.03 0.035 0.045"/>
+        </geometry>
+        <origin xyz="0.0 0.0 0.0" rpy="0 0 0" />
+        <material name="blue">
+            <color rgba="0 0 0.8 1"/>
+        </material>
+      </visual>
+    </link>
+    <joint name="arm_waist_joint" type="revolute">
+      <axis xyz="0 0 1"/>
+      <limit effort="1000.0" lower="-3.1416" upper="3.1416" velocity="0.5"/>
+      <origin xyz="0.0 0.0 0.035" rpy="0 0 0" />
+      <parent link="arm_base_link"/>
+      <child link="arm_waist_link" />
+    </joint>
+    <link name="arm_shoulder_link">
+      <visual>
+        <geometry>
+          <box size="0.025 0.045 0.05"/>
+        </geometry>
+        <origin xyz="0.0 0.0 0.0" rpy="0 0 0" />
+        <material name="white">
+            <color rgba="1 1 1 1"/>
+        </material>
+      </visual>
+    </link>
+    <joint name="arm_shoulder_joint" type="revolute">
+      <axis xyz="0 1 0"/>
+      <limit effort="1000.0" lower="-3.1416" upper="3.1416" velocity="0.5"/>
+      <origin xyz="0.00 0.00 0.045" rpy="0 0 0.0" />
+      <parent link="arm_waist_link"/>
+      <child link="arm_shoulder_link" />
+    </joint>
     <!-- Kobuki Gazebo simulation details -->
     <kobuki_sim/>

Commit message: elbow added to tf_motors

File: common/kobuki.urdf.xacro (robot description, xacro)
@@ -275,22 +275,22 @@
         </geometry>
         <origin xyz="0.0 0.0 0.0" rpy="0 0 0" />
+        <material name="blue">
+            <color rgba="0 0 0.8 1"/>
+        </material>
+      </visual>
+    </link>
+    <joint name="arm_base_joint" type="fixed">
+      <origin xyz="0.10 0.00 0.27" rpy="0 0 0" />
+      <parent link="base_link"/>
+      <child link="arm_base_link" />
+    </joint>
+    <link name="arm_waist_link">
+      <visual>
+        <geometry>
+          <box size="0.03 0.035 0.045"/>
+        </geometry>
+        <origin xyz="0.0 0.0 0.0" rpy="0 0 0" />
         <material name="black">
             <color rgba="0 0 0 1"/>
-        </material>
-      </visual>
-    </link>
-    <joint name="arm_base_joint" type="fixed">
-      <origin xyz="0.10 0.00 0.27" rpy="0 0 0" />
-      <parent link="base_link"/>
-      <child link="arm_base_link" />
-    </joint>
-    <link name="arm_waist_link">
-      <visual>
-        <geometry>
-          <box size="0.03 0.035 0.045"/>
-        </geometry>
-        <origin xyz="0.0 0.0 0.0" rpy="0 0 0" />
-        <material name="blue">
-            <color rgba="0 0 0.8 1"/>
         </material>
       </visual>
@@ -317,7 +317,41 @@
       <axis xyz="0 1 0"/>
       <limit effort="1000.0" lower="-3.1416" upper="3.1416" velocity="0.5"/>
-      <origin xyz="0.00 0.00 0.045" rpy="0 0 0.0" />
+      <origin xyz="0.00 0.00 0.035" rpy="0 0 0.0" />
       <parent link="arm_waist_link"/>
       <child link="arm_shoulder_link" />
+    </joint>
+    <link name="arm_elbow_base_link">
+      <visual>
+        <geometry>
+          <box size="0.03 0.035 0.045"/>
+        </geometry>
+        <origin xyz="0.0 0.0 0.0" rpy="0 0 0" />
+        <material name="black">
+            <color rgba="0 0 0 1"/>
+        </material>
+      </visual>
+    </link>
+    <joint name="arm_elbow_base_joint" type="fixed">
+      <origin xyz="0.0 0.00 0.045" rpy="0 0 0" />
+      <parent link="arm_shoulder_link"/>
+      <child link="arm_elbow_base_link" />
+    </joint>
+    <link name="arm_elbow_link">
+      <visual>
+        <geometry>
+          <box size="0.025 0.045 0.05"/>
+        </geometry>
+        <origin xyz="0.0 0.0 0.0" rpy="0 0 0" />
+        <material name="white">
+            <color rgba="1 1 1 1"/>
+        </material>
+      </visual>
+    </link>
+    <joint name="arm_elbow_joint" type="revolute">
+      <axis xyz="0 1 0"/>
+      <limit effort="1000.0" lower="-3.1416" upper="3.1416" velocity="0.5"/>
+      <origin xyz="0.00 0.00 0.045" rpy="0 0 0.0" />
+      <parent link="arm_elbow_base_link"/>
+      <child link="arm_elbow_link" />
     </joint>
     <!-- Kobuki Gazebo simulation details -->

Commit message: wrist added to tf_motors

File: common/kobuki.urdf.xacro (robot description, xacro)
@@ -281,5 +281,5 @@
     </link>
     <joint name="arm_base_joint" type="fixed">
-      <origin xyz="0.10 0.00 0.27" rpy="0 0 0" />
+      <origin xyz="0.10 0.00 0.45" rpy="0 0 0" />
       <parent link="base_link"/>
       <child link="arm_base_link" />
@@ -333,5 +333,5 @@
     </link>
     <joint name="arm_elbow_base_joint" type="fixed">
-      <origin xyz="0.0 0.00 0.045" rpy="0 0 0" />
+      <origin xyz="0.0 0.00 0.05" rpy="0 0 0" />
       <parent link="arm_shoulder_link"/>
       <child link="arm_elbow_base_link" />
@@ -354,4 +354,38 @@
       <parent link="arm_elbow_base_link"/>
       <child link="arm_elbow_link" />
+    </joint>
+    <link name="arm_wrist_base_link">
+      <visual>
+        <geometry>
+          <box size="0.03 0.035 0.045"/>
+        </geometry>
+        <origin xyz="0.0 0.0 0.0" rpy="0 0 0" />
+        <material name="black">
+            <color rgba="0 0 0 1"/>
+        </material>
+      </visual>
+    </link>
+    <joint name="arm_wrist_base_joint" type="fixed">
+      <origin xyz="0.0 0.00 0.05" rpy="0 0 0" />
+      <parent link="arm_elbow_link"/>
+      <child link="arm_wrist_base_link" />
+    </joint>
+    <link name="arm_wrist_link">
+      <visual>
+        <geometry>
+          <box size="0.025 0.045 0.05"/>
+        </geometry>
+        <origin xyz="0.0 0.0 0.0" rpy="0 0 0" />
+        <material name="white">
+            <color rgba="1 1 1 1"/>
+        </material>
+      </visual>
+    </link>
+    <joint name="arm_wrist_joint" type="revolute">
+      <axis xyz="0 1 0"/>
+      <limit effort="1000.0" lower="-3.1416" upper="3.1416" velocity="0.5"/>
+      <origin xyz="0.00 0.00 0.045" rpy="0 0 0.0" />
+      <parent link="arm_wrist_base_link"/>
+      <child link="arm_wrist_link" />
     </joint>
     <!-- Kobuki Gazebo simulation details -->

Commit message: hand added to tf_motors

File: common/kobuki.urdf.xacro (robot description, xacro)
@@ -210,28 +210,30 @@
     <!-- FEATURED ROBOT MODEL -->
     <!-- head pan_tilt -->
+    <!-- head base -->
     <link name="head_base_link">
       <visual>
         <geometry>
           <box size="0.045 0.03 0.035"/>
+        </geometry>
+        <origin xyz="0.0 0.0 0.0" rpy="0 0 0" />
+        <material name="blue">
+            <color rgba="0 0 0.8 1"/>
+        </material>
+      </visual>
+    </link>
+    <joint name="head_base_joint" type="fixed">
+      <origin xyz="-0.20 0.00 0.90" rpy="0 0 0" />
+      <parent link="base_link"/>
+      <child link="head_base_link" />
+    </joint>
+    <!-- head pan -->
+    <link name="head_pan_link">
+      <visual>
+        <geometry>
+          <box size="0.03 0.035 0.045"/>
         </geometry>
         <origin xyz="0.0 0.0 0.0" rpy="0 0 0" />
         <material name="black">
             <color rgba="0 0 0 1"/>
-        </material>
-      </visual>
-    </link>
-    <joint name="head_base_joint" type="fixed">
-      <origin xyz="-0.20 0.00 0.90" rpy="0 0 0" />
-      <parent link="base_link"/>
-      <child link="head_base_link" />
-    </joint>
-    <link name="head_pan_link">
-      <visual>
-        <geometry>
-          <box size="0.03 0.035 0.045"/>
-        </geometry>
-        <origin xyz="0.0 0.0 0.0" rpy="0 0 0" />
-        <material name="blue">
-            <color rgba="0 0 0.8 1"/>
         </material>
       </visual>
@@ -244,4 +246,5 @@
       <child link="head_pan_link" />
     </joint>
+    <!-- head tilt -->
     <link name="head_tilt_link">
       <visual>
@@ -258,8 +261,9 @@
       <axis xyz="0 1 0"/>
       <limit effort="1000.0" lower="-3.1416" upper="3.1416" velocity="0.5"/>
-      <origin xyz="0.00 0.00 0.045" rpy="0 0 0.0" />
+      <origin xyz="0.00 0.00 0.045" rpy="0 0 0" />
       <parent link="head_pan_link"/>
       <child link="head_tilt_link" />
     </joint>
+    <!-- camera -->
     <link name="camera_rgb_frame"/>
     <joint name="camera_rgb_joint" type="fixed">
@@ -269,4 +273,5 @@
     </joint>
     <!-- robot arm as in built as in http://wiki.ros.org/turtlebot_arm -->
+    <!-- arm base -->
     <link name="arm_base_link">
       <visual>
@@ -281,8 +286,9 @@
     </link>
     <joint name="arm_base_joint" type="fixed">
-      <origin xyz="0.10 0.00 0.45" rpy="0 0 0" />
+      <origin xyz="0.10 0.00 0.40" rpy="0 0 0" />
       <parent link="base_link"/>
       <child link="arm_base_link" />
     </joint>
+    <!-- arm waist -->
     <link name="arm_waist_link">
       <visual>
@@ -303,4 +309,5 @@
       <child link="arm_waist_link" />
     </joint>
+    <!-- arm shoulder -->
     <link name="arm_shoulder_link">
       <visual>
@@ -317,8 +324,9 @@
       <axis xyz="0 1 0"/>
       <limit effort="1000.0" lower="-3.1416" upper="3.1416" velocity="0.5"/>
-      <origin xyz="0.00 0.00 0.035" rpy="0 0 0.0" />
+      <origin xyz="0.00 0.00 0.035" rpy="0 0 0" />
       <parent link="arm_waist_link"/>
       <child link="arm_shoulder_link" />
     </joint>
+    <!-- arm elbow -->
     <link name="arm_elbow_base_link">
       <visual>
@@ -351,8 +359,9 @@
       <axis xyz="0 1 0"/>
       <limit effort="1000.0" lower="-3.1416" upper="3.1416" velocity="0.5"/>
-      <origin xyz="0.00 0.00 0.045" rpy="0 0 0.0" />
+      <origin xyz="0.00 0.00 0.045" rpy="0 0 0" />
       <parent link="arm_elbow_base_link"/>
       <child link="arm_elbow_link" />
     </joint>
+    <!-- arm wrist -->
     <link name="arm_wrist_base_link">
       <visual>
@@ -374,5 +383,5 @@
       <visual>
         <geometry>
-          <box size="0.025 0.045 0.05"/>
+          <box size="0.025 0.045 0.025"/>
         </geometry>
         <origin xyz="0.0 0.0 0.0" rpy="0 0 0" />
@@ -385,7 +394,26 @@
       <axis xyz="0 1 0"/>
       <limit effort="1000.0" lower="-3.1416" upper="3.1416" velocity="0.5"/>
-      <origin xyz="0.00 0.00 0.045" rpy="0 0 0.0" />
+      <origin xyz="0.00 0.00 0.045" rpy="0 0 0" />
       <parent link="arm_wrist_base_link"/>
       <child link="arm_wrist_link" />
+    </joint>
+    <!-- arm hand -->
+    <link name="arm_hand_link">
+      <visual>
+        <geometry>
+          <box size="0.035 0.045 0.03"/>
+        </geometry>
+        <origin xyz="0.0 0.0 0.0" rpy="0 0 0" />
+        <material name="white">
+            <color rgba="1 1 1 1"/>
+        </material>
+      </visual>
+    </link>
+    <joint name="arm_hand_joint" type="revolute">
+      <axis xyz="0 1 0"/>
+      <limit effort="1000.0" lower="-3.1416" upper="3.1416" velocity="0.5"/>
+      <origin xyz="0.00 0.00 0.025" rpy="0 1.57 1.57" />
+      <parent link="arm_wrist_link"/>
+      <child link="arm_hand_link" />
     </joint>
     <!-- Kobuki Gazebo simulation details -->

Commit message: hand added to tf_motors fixed

File: common/kobuki.urdf.xacro (robot description, xacro)
@@ -402,5 +402,5 @@
       <visual>
         <geometry>
-          <box size="0.035 0.045 0.03"/>
+          <box size="0.03 0.035 0.045"/>
         </geometry>
         <origin xyz="0.0 0.0 0.0" rpy="0 0 0" />

Commit message: hand added to tf_motors fixed

File: common/kobuki.urdf.xacro (robot description, xacro)
@@ -399,10 +399,26 @@
     </joint>
     <!-- arm hand -->
+    <link name="arm_hand_base_link">
+      <visual>
+        <geometry>
+          <box size="0.03 0.035 0.045"/>
+        </geometry>
+        <origin xyz="0.0 0.0 0.0" rpy="0 0 0" />
+        <material name="black">
+            <color rgba="0 0 0 1"/>
+        </material>
+      </visual>
+    </link>
+    <joint name="arm_hand_base_joint" type="fixed">
+      <origin xyz="0.0 0.00 0.025" rpy="0 0 0" />
+      <parent link="arm_wrist_link"/>
+      <child link="arm_hand_base_link" />
+    </joint>
     <link name="arm_hand_link">
       <visual>
         <geometry>
-          <box size="0.03 0.035 0.045"/>
-        </geometry>
-        <origin xyz="0.0 0.0 0.0" rpy="0 0 0" />
+          <box size="0.03 0.05 0.005"/>
+        </geometry>
+        <origin xyz="0.0 0.0 0.0" rpy="0 1.57 1.57" />
         <material name="white">
             <color rgba="1 1 1 1"/>
@@ -413,6 +429,6 @@
       <axis xyz="0 1 0"/>
       <limit effort="1000.0" lower="-3.1416" upper="3.1416" velocity="0.5"/>
-      <origin xyz="0.00 0.00 0.025" rpy="0 1.57 1.57" />
-      <parent link="arm_wrist_link"/>
+      <origin xyz="0.00 0.00 0.045" rpy="0 1.57 1.57" />
+      <parent link="arm_hand_base_link"/>
       <child link="arm_hand_link" />
     </joint>

Commit message: hand added to tf_motors fixed

File: common/kobuki.urdf.xacro (robot description, xacro)
@@ -286,5 +286,5 @@
     </link>
     <joint name="arm_base_joint" type="fixed">
-      <origin xyz="0.10 0.00 0.40" rpy="0 0 0" />
+      <origin xyz="0.10 0.00 0.43" rpy="0 0 0" />
       <parent link="base_link"/>
       <child link="arm_base_link" />
@@ -418,5 +418,5 @@
       <visual>
         <geometry>
-          <box size="0.03 0.05 0.005"/>
+          <box size="0.005 0.05 0.03"/>
         </geometry>
         <origin xyz="0.0 0.0 0.0" rpy="0 1.57 1.57" />
