Commit message: palm link added

File: common/kobuki.urdf.xacro (robot description, xacro)
@@ -433,4 +433,20 @@
       <child link="arm_hand_link" />
     </joint>
+    <link name="arm_hand_palm_link">
+      <visual>
+        <geometry>
+          <box size="0.005 0.05 0.03"/>
+        </geometry>
+        <origin xyz="0.0 0.0 0.045" rpy="0 1.57 1.57" />
+        <material name="white">
+            <color rgba="1 1 1 1"/>
+        </material>
+      </visual>
+    </link>
+    <joint name="arm_hand_joint" type="fixed">
+      <origin xyz="0.00 0.00 0.045" rpy="0 1.57 1.57" />
+      <parent link="arm_hand_base_link"/>
+      <child link="arm_hand_palm_link" />
+    </joint>
     <!-- Kobuki Gazebo simulation details -->
     <kobuki_sim/>

Commit message: palm link fixed

File: common/kobuki.urdf.xacro (robot description, xacro)
@@ -444,5 +444,5 @@
       </visual>
     </link>
-    <joint name="arm_hand_joint" type="fixed">
+    <joint name="arm_hand_palm_joint" type="fixed">
       <origin xyz="0.00 0.00 0.045" rpy="0 1.57 1.57" />
       <parent link="arm_hand_base_link"/>

Commit message: 3d model fixed

File: common/kobuki.urdf.xacro (robot description, xacro)
@@ -242,5 +242,5 @@
       <axis xyz="0 0 1"/>
       <limit effort="1000.0" lower="-3.1416" upper="3.1416" velocity="0.5"/>
-      <origin xyz="0.0 0.0 0.035" rpy="0 0 0" />
+      <origin xyz="0.0 0.0 0.040" rpy="0 0 0" />
       <parent link="head_base_link"/>
       <child link="head_pan_link" />
@@ -261,5 +261,5 @@
       <axis xyz="0 1 0"/>
       <limit effort="1000.0" lower="-3.1416" upper="3.1416" velocity="0.5"/>
-      <origin xyz="0.00 0.00 0.045" rpy="0 0 0" />
+      <origin xyz="0.00 0.00 0.0475" rpy="0 0 0" />
       <parent link="head_pan_link"/>
       <child link="head_tilt_link" />
@@ -305,5 +305,5 @@
       <axis xyz="0 0 1"/>
       <limit effort="1000.0" lower="-3.1416" upper="3.1416" velocity="0.5"/>
-      <origin xyz="0.0 0.0 0.035" rpy="0 0 0" />
+      <origin xyz="0.0 0.0 0.040" rpy="0 0 0" />
       <parent link="arm_base_link"/>
       <child link="arm_waist_link" />
@@ -324,5 +324,5 @@
       <axis xyz="0 1 0"/>
       <limit effort="1000.0" lower="-3.1416" upper="3.1416" velocity="0.5"/>
-      <origin xyz="0.00 0.00 0.035" rpy="0 0 0" />
+      <origin xyz="0.00 0.00 0.0475" rpy="0 0 0" />
       <parent link="arm_waist_link"/>
       <child link="arm_shoulder_link" />
@@ -341,5 +341,5 @@
     </link>
     <joint name="arm_elbow_base_joint" type="fixed">
-      <origin xyz="0.0 0.00 0.05" rpy="0 0 0" />
+      <origin xyz="0.0 0.00 0.0475" rpy="0 0 0" />
       <parent link="arm_shoulder_link"/>
       <child link="arm_elbow_base_link" />
@@ -359,5 +359,5 @@
       <axis xyz="0 1 0"/>
       <limit effort="1000.0" lower="-3.1416" upper="3.1416" velocity="0.5"/>
-      <origin xyz="0.00 0.00 0.045" rpy="0 0 0" />
+      <origin xyz="0.00 0.00 0.0475" rpy="0 0 0" />
       <parent link="arm_elbow_base_link"/>
       <child link="arm_elbow_link" />
@@ -376,5 +376,5 @@
     </link>
     <joint name="arm_wrist_base_joint" type="fixed">
-      <origin xyz="0.0 0.00 0.05" rpy="0 0 0" />
+      <origin xyz="0.0 0.00 0.0475" rpy="0 0 0" />
       <parent link="arm_elbow_link"/>
       <child link="arm_wrist_base_link" />
@@ -394,5 +394,5 @@
       <axis xyz="0 1 0"/>
       <limit effort="1000.0" lower="-3.1416" upper="3.1416" velocity="0.5"/>
-      <origin xyz="0.00 0.00 0.045" rpy="0 0 0" />
+      <origin xyz="0.00 0.00 0.035" rpy="0 0 0" />
       <parent link="arm_wrist_base_link"/>
       <child link="arm_wrist_link" />
@@ -402,5 +402,5 @@
       <visual>
         <geometry>
-          <box size="0.03 0.035 0.045"/>
+          <box size="0.035 0.045 0.03"/>
         </geometry>
         <origin xyz="0.0 0.0 0.0" rpy="0 0 0" />
@@ -411,5 +411,5 @@
     </link>
     <joint name="arm_hand_base_joint" type="fixed">
-      <origin xyz="0.0 0.00 0.025" rpy="0 0 0" />
+      <origin xyz="0.0 0.00 0.035" rpy="0 0 0" />
       <parent link="arm_wrist_link"/>
       <child link="arm_hand_base_link" />
@@ -429,5 +429,5 @@
       <axis xyz="0 1 0"/>
       <limit effort="1000.0" lower="-3.1416" upper="3.1416" velocity="0.5"/>
-      <origin xyz="0.00 0.00 0.045" rpy="0 1.57 1.57" />
+      <origin xyz="0.00 -0.0225 0.03" rpy="0 1.57 1.57" />
       <parent link="arm_hand_base_link"/>
       <child link="arm_hand_link" />
@@ -438,5 +438,5 @@
           <box size="0.005 0.05 0.03"/>
         </geometry>
-        <origin xyz="0.0 0.0 0.045" rpy="0 1.57 1.57" />
+        <origin xyz="0.0 0.0 0.0" rpy="0 1.57 1.57" />
         <material name="white">
             <color rgba="1 1 1 1"/>
@@ -445,5 +445,5 @@
     </link>
     <joint name="arm_hand_palm_joint" type="fixed">
-      <origin xyz="0.00 0.00 0.045" rpy="0 1.57 1.57" />
+      <origin xyz="0.00 0.0225 0.03" rpy="0 1.57 1.57" />
       <parent link="arm_hand_base_link"/>
       <child link="arm_hand_palm_link" />

Commit message: 3d model fixed

File: common/kobuki.urdf.xacro (robot description, xacro)
@@ -411,5 +411,5 @@
     </link>
     <joint name="arm_hand_base_joint" type="fixed">
-      <origin xyz="0.0 0.00 0.035" rpy="0 0 0" />
+      <origin xyz="0.0 0.00 0.0275" rpy="0 0 0" />
       <parent link="arm_wrist_link"/>
       <child link="arm_hand_base_link" />
@@ -436,5 +436,5 @@
       <visual>
         <geometry>
-          <box size="0.005 0.05 0.03"/>
+          <box size="0.005 0.04 0.03"/>
         </geometry>
         <origin xyz="0.0 0.0 0.0" rpy="0 1.57 1.57" />

Commit message: 3d model fixed

File: common/kobuki.urdf.xacro (robot description, xacro)
@@ -429,5 +429,5 @@
       <axis xyz="0 1 0"/>
       <limit effort="1000.0" lower="-3.1416" upper="3.1416" velocity="0.5"/>
-      <origin xyz="0.00 -0.0225 0.03" rpy="0 1.57 1.57" />
+      <origin xyz="0.00 -0.0225 0.04" rpy="0 1.57 1.57" />
       <parent link="arm_hand_base_link"/>
       <child link="arm_hand_link" />
@@ -445,5 +445,5 @@
     </link>
     <joint name="arm_hand_palm_joint" type="fixed">
-      <origin xyz="0.00 0.0225 0.03" rpy="0 1.57 1.57" />
+      <origin xyz="0.00 0.0225 0.035" rpy="0 1.57 1.57" />
       <parent link="arm_hand_base_link"/>
       <child link="arm_hand_palm_link" />

Commit message: head tilt link updated

File: common/kobuki.urdf.xacro (robot description, xacro)
@@ -250,5 +250,5 @@
       <visual>
         <geometry>
-          <box size="0.025 0.045 0.05"/>
+          <box size="0.025 0.045 0.025"/>
         </geometry>
         <origin xyz="0.0 0.0 0.0" rpy="0 0 0" />
@@ -261,5 +261,5 @@
       <axis xyz="0 1 0"/>
       <limit effort="1000.0" lower="-3.1416" upper="3.1416" velocity="0.5"/>
-      <origin xyz="0.00 0.00 0.0475" rpy="0 0 0" />
+      <origin xyz="0.00 0.00 0.035" rpy="0 0 0" />
       <parent link="head_pan_link"/>
       <child link="head_tilt_link" />

Commit message: head tilt link updated

File: common/kobuki.urdf.xacro (robot description, xacro)
@@ -268,5 +268,5 @@
     <link name="camera_rgb_frame"/>
     <joint name="camera_rgb_joint" type="fixed">
-      <origin xyz="0.0 0.0 0.05" rpy="0 0 0" />
+      <origin xyz="0.0 0.0 0.025" rpy="0 0 0" />
       <parent link="head_tilt_link"/>
       <child link="camera_rgb_frame" />

Commit message: head tilt link updated

File: common/kobuki.urdf.xacro (robot description, xacro)
@@ -268,5 +268,5 @@
     <link name="camera_rgb_frame"/>
     <joint name="camera_rgb_joint" type="fixed">
-      <origin xyz="0.0 0.0 0.025" rpy="0 0 0" />
+      <origin xyz="0.0 0.0 0.035" rpy="0 0 0" />
       <parent link="head_tilt_link"/>
       <child link="camera_rgb_frame" />

Commit message: head tilt link updated

File: common/kobuki.urdf.xacro (robot description, xacro)
@@ -268,5 +268,5 @@
     <link name="camera_rgb_frame"/>
     <joint name="camera_rgb_joint" type="fixed">
-      <origin xyz="0.0 0.0 0.035" rpy="0 0 0" />
+      <origin xyz="0.0 0.0 0.04" rpy="0 0 0" />
       <parent link="head_tilt_link"/>
       <child link="camera_rgb_frame" />
